File: FSKmodem/FSKmodem.kicad_sch (KiCad schematic)
At the start: 9 parts, among them IC1 TCM3105, Q1 CSTLS_G

Commit message: ready for lut
Connections:
- no-connect marks 0 -> 3
Changed lines of the file:
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@@
   (junction (at 147.32 132.08) (diameter 0) (color 0 0 0 0)
   )
+  (no_connect (at 157.48 99.06))
+  (no_connect (at 137.16 91.44))
+  (no_connect (at 137.16 104.14))
   (wire (pts (xy 180.34 96.52) (xy 177.8 96.52))
     (stroke (width 0.1524) (type solid))
